File: A_BACKPLATES/A02/A02.kicad_pcb (KiCad board)
At the start: 2 copper layers, 183 x 110 mm, 218 parts, among them J0 Conn_01x01_Male, J1 Conn_01x01_Male, J2 Conn_01x01_Male, J3 Conn_01x01_Male

Commit message: A02 all mounting holes placed
Parts:
- removed HE16, HF10, HF17, HF7, HH17, HJ10, HJ7: MountingHole, MountingHole:MountingHole_3mm
- moved J0 229.0 mm to (-3.73, 59.7)
- moved J1 222.3 mm to (-3.81, 86.5)
- moved HZ7 195.7 mm to (51.7, 29.1)
- moved HZ8 181.8 mm to (51.7, 120.1)
- moved HZ10 180.5 mm to (73.7, 120.6)
- moved HZ9 154.1 mm to (73.7, 28.6)
- moved HZ13 148.1 mm to (92.7, 116.6)
- moved HZ14 126.0 mm to (127.7, 116.6)
- moved HZ12 125.8 mm to (92.7, 74.6)
- moved HZ11 123.5 mm to (127.7, 74.6)
- moved HZ15 100.0 mm to (150.7, 28.6)
- moved HZ19 58.2 mm to (197.7, 94.6)
- moved HZ20 52.7 mm to (191.7, 120.1)
- moved J2 51.7 mm to (212.5, 55.9)
- moved HZ16 42.7 mm to (191.7, 29.1)
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Changed lines of the file:
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@@
     (tracks 0)
     (zones 0)
-    (modules 218)
+    (modules 211)
     (nets 2)
   )
@@
   )
   (module MountingHole:MountingHole_3mm (layer F.Cu)
-    (at 216.8398 73.8632)
+    (at 191.67 120.11)
     (descr "Mounting Hole 3mm, no annular")
     (tags "mounting hole 3mm no annular")
@@
   )
   (module MountingHole:MountingHole_3mm (layer F.Cu)
-    (at 247.1674 64.0334)
+    (at 197.67 94.61)
     (descr "Mounting Hole 3mm, no annular")
     (tags "mounting hole 3mm no annular")
@@
   )
   (module MountingHole:MountingHole_3mm (layer F.Cu)
-    (at 236.7788 63.9572)
+    (at 197.67 74.61)
     (descr "Mounting Hole 3mm, no annular")
     (tags "mounting hole 3mm no annular")
@@
   )
   (module MountingHole:MountingHole_3mm (layer F.Cu)
-    (at 226.8728 63.9572)
+    (at 189.67 62.61)
     (descr "Mounting Hole 3mm, no annular")
     (tags "mounting hole 3mm no annular")
@@
   )
   (module MountingHole:MountingHole_3mm (layer F.Cu)
-    (at 216.8398 63.6016)
+    (at 191.67 29.11)
     (descr "Mounting Hole 3mm, no annular")
     (tags "mounting hole 3mm no annular")
@@
   )
   (module Connector_Wire:SolderWirePad_1x01_Drill1mm (layer F.Cu)
-    (at 231.14 117.475)
+    (at 212.5472 83.4644)
     (descr "Wire solder connection")
     (tags connector)
@@
   )
   (module Connector_Wire:SolderWirePad_1x01_Drill1mm (layer F.Cu)
-    (at 231.14 104.14)
+    (at 212.5472 55.9054)
     (descr "Wire solder connection")
     (tags connector)
@@
   )
   (module Connector_Wire:SolderWirePad_1x01_Drill1mm (layer F.Cu)
-    (at 217.805 104.14)
+    (at -3.81 86.5378)
     (descr "Wire solder connection")
     (tags connector)
@@
   )
   (module Connector_Wire:SolderWirePad_1x01_Drill1mm (layer F.Cu)
-    (at 217.805 117.475)
+    (at -3.7338 59.69)
     (descr "Wire solder connection")
     (tags connector)
@@
   )
   (module MountingHole:MountingHole_3mm (layer F.Cu)
-    (at 247.33 54.29)
+    (at 150.67 28.61)
     (descr "Mounting Hole 3mm, no annular")
     (tags "mounting hole 3mm no annular")
@@
   )
   (module MountingHole:MountingHole_3mm (layer F.Cu)
-    (at 237.17 54.29)
+    (at 127.67 116.61)
     (descr "Mounting Hole 3mm, no annular")
     (tags "mounting hole 3mm no annular")
@@
   )
   (module MountingHole:MountingHole_3mm (layer F.Cu)
-    (at 227.01 54.29)
+    (at 92.67 116.61)
     (descr "Mounting Hole 3mm, no annular")
     (tags "mounting hole 3mm no annular")
@@
   )
   (module MountingHole:MountingHole_3mm (layer F.Cu)
-    (at 216.85 54.29)
+    (at 92.67 74.61)
     (descr "Mounting Hole 3mm, no annular")
     (tags "mounting hole 3mm no annular")
@@
   )
   (module MountingHole:MountingHole_3mm (layer F.Cu)
-    (at 247.33 44.13)
+    (at 127.67 74.61)
     (descr "Mounting Hole 3mm, no annular")
     (tags "mounting hole 3mm no annular")
@@
   )
   (module MountingHole:MountingHole_3mm (layer F.Cu)
-    (at 237.17 44.13)
+    (at 73.67 120.61)
     (descr "Mounting Hole 3mm, no annular")
     (tags "mounting hole 3mm no annular")
@@
   )
   (module MountingHole:MountingHole_3mm (layer F.Cu)
-    (at 227.01 44.13)
+    (at 73.67 28.61)
     (descr "Mounting Hole 3mm, no annular")
     (tags "mounting hole 3mm no annular")
@@
   )
   (module MountingHole:MountingHole_3mm (layer F.Cu)
-    (at 216.85 44.13)
+    (at 51.67 120.11)
     (descr "Mounting Hole 3mm, no annular")
     (tags "mounting hole 3mm no annular")
@@
   )
   (module MountingHole:MountingHole_3mm (layer F.Cu)
-    (at 247.33 33.97)
+    (at 51.67 29.11)
     (descr "Mounting Hole 3mm, no annular")
     (tags "mounting hole 3mm no annular")
@@
   )
   (module MountingHole:MountingHole_3mm (layer F.Cu)
-    (at 125.41 115.25)
-    (descr "Mounting Hole 3mm, no annular")
-    (tags "mounting hole 3mm no annular")
-    (attr virtual)
-    (fp_text reference HJ10 (at 0 -4) (layer F.SilkS) hide
-      (effects (font (size 1 1) (thickness 0.15)))
-    )
-    (fp_text value MountingHole (at 0 4) (layer F.Fab)
-      (effects (font (size 1 1) (thickness 0.15)))
-    )
-    (fp_circle (center 0 0) (end 3.25 0) (layer F.CrtYd) (width 0.05))
-    (fp_circle (center 0 0) (end 3 0) (layer Cmts.User) (width 0.15))
-    (fp_text user %R (at 0.3 0) (layer F.Fab)
-      (effects (font (size 1 1) (thickness 0.15)))
-    )
-    (pad 1 np_thru_hole circle (at 0 0) (size 3 3) (drill 3) (layers *.Cu *.Mask))
-  )
-  (module MountingHole:MountingHole_3mm (layer F.Cu)
     (at 115.25 115.25)
     (descr "Mounting Hole 3mm, no annular")
@@
   )
   (module MountingHole:MountingHole_3mm (layer F.Cu)
-    (at 94.93 115.25)
-    (descr "Mounting Hole 3mm, no annular")
-    (tags "mounting hole 3mm no annular")
-    (attr virtual)
-    (fp_text reference HJ7 (at 0 -4) (layer F.SilkS) hide
-      (effects (font (size 1 1) (thickness 0.15)))
-    )
-    (fp_text value MountingHole (at 0 4) (layer F.Fab)
-      (effects (font (size 1 1) (thickness 0.15)))
-    )
-    (fp_circle (center 0 0) (end 3.25 0) (layer F.CrtYd) (width 0.05))
-    (fp_circle (center 0 0) (end 3 0) (layer Cmts.User) (width 0.15))
-    (fp_text user %R (at 0.3 0) (layer F.Fab)
-      (effects (font (size 1 1) (thickness 0.15)))
-    )
-    (pad 1 np_thru_hole circle (at 0 0) (size 3 3) (drill 3) (layers *.Cu *.Mask))
-  )
-  (module MountingHole:MountingHole_3mm (layer F.Cu)
     (at 84.77 115.25)
     (descr "Mounting Hole 3mm, no annular")
@@
   )
   (module MountingHole:MountingHole_3mm (layer F.Cu)
-    (at 196.53 94.93)
-    (descr "Mounting Hole 3mm, no annular")
-    (tags "mounting hole 3mm no annular")
-    (attr virtual)
-    (fp_text reference HH17 (at 0 -4) (layer F.SilkS) hide
-      (effects (font (size 1 1) (thickness 0.15)))
-    )
-    (fp_text value MountingHole (at 0 4) (layer F.Fab)
-      (effects (font (size 1 1) (thickness 0.15)))
-    )
-    (fp_circle (center 0 0) (end 3.25 0) (layer F.CrtYd) (width 0.05))
-    (fp_circle (center 0 0) (end 3 0) (layer Cmts.User) (width 0.15))
-    (fp_text user %R (at 0.3 0) (layer F.Fab)
-      (effects (font (size 1 1) (thickness 0.15)))
-    )
-    (pad 1 np_thru_hole circle (at 0 0) (size 3 3) (drill 3) (layers *.Cu *.Mask))
-  )
-  (module MountingHole:MountingHole_3mm (layer F.Cu)
     (at 186.37 94.93)
     (descr "Mounting Hole 3mm, no annular")
@@
   )
   (module MountingHole:MountingHole_3mm (layer F.Cu)
-    (at 196.53 74.61)
-    (descr "Mounting Hole 3mm, no annular")
-    (tags "mounting hole 3mm no annular")
-    (attr virtual)
-    (fp_text reference HF17 (at 0 -4) (layer F.SilkS) hide
-      (effects (font (size 1 1) (thickness 0.15)))
-    )
-    (fp_text value MountingHole (at 0 4) (layer F.Fab)
-      (effects (font (size 1 1) (thickness 0.15)))
-    )
-    (fp_circle (center 0 0) (end 3.25 0) (layer F.CrtYd) (width 0.05))
-    (fp_circle (center 0 0) (end 3 0) (layer Cmts.User) (width 0.15))
-    (fp_text user %R (at 0.3 0) (layer F.Fab)
-      (effects (font (size 1 1) (thickness 0.15)))
-    )
-    (pad 1 np_thru_hole circle (at 0 0) (size 3 3) (drill 3) (layers *.Cu *.Mask))
-  )
-  (module MountingHole:MountingHole_3mm (layer F.Cu)
     (at 186.37 74.61)
     (descr "Mounting Hole 3mm, no annular")
@@
   )
   (module MountingHole:MountingHole_3mm (layer F.Cu)
-    (at 125.41 74.61)
-    (descr "Mounting Hole 3mm, no annular")
-    (tags "mounting hole 3mm no annular")
-    (attr virtual)
-    (fp_text reference HF10 (at 0 -4) (layer F.SilkS) hide
-      (effects (font (size 1 1) (thickness 0.15)))
-    )
-    (fp_text value MountingHole (at 0 4) (layer F.Fab)
-      (effects (font (size 1 1) (thickness 0.15)))
-    )
-    (fp_circle (center 0 0) (end 3.25 0) (layer F.CrtYd) (width 0.05))
-    (fp_circle (center 0 0) (end 3 0) (layer Cmts.User) (width 0.15))
-    (fp_text user %R (at 0.3 0) (layer F.Fab)
-      (effects (font (size 1 1) (thickness 0.15)))
-    )
-    (pad 1 np_thru_hole circle (at 0 0) (size 3 3) (drill 3) (layers *.Cu *.Mask))
-  )
-  (module MountingHole:MountingHole_3mm (layer F.Cu)
     (at 115.25 74.61)
     (descr "Mounting Hole 3mm, no annular")
@@
   )
   (module MountingHole:MountingHole_3mm (layer F.Cu)
-    (at 94.93 74.61)
-    (descr "Mounting Hole 3mm, no annular")
-    (tags "mounting hole 3mm no annular")
-    (attr virtual)
-    (fp_text reference HF7 (at 0 -4) (layer F.SilkS) hide
-      (effects (font (size 1 1) (thickness 0.15)))
-    )
-    (fp_text value MountingHole (at 0 4) (layer F.Fab)
-      (effects (font (size 1 1) (thickness 0.15)))
-    )
-    (fp_circle (center 0 0) (end 3.25 0) (layer F.CrtYd) (width 0.05))
-    (fp_circle (center 0 0) (end 3 0) (layer Cmts.User) (width 0.15))
-    (fp_text user %R (at 0.3 0) (layer F.Fab)
-      (effects (font (size 1 1) (thickness 0.15)))
-    )
-    (pad 1 np_thru_hole circle (at 0 0) (size 3 3) (drill 3) (layers *.Cu *.Mask))
-  )
-  (module MountingHole:MountingHole_3mm (layer F.Cu)
     (at 84.77 74.61)
     (descr "Mounting Hole 3mm, no annular")
@@
       (effects (font (size 1 1) (thickness 0.15)))
     )
-    (fp_text value MountingHole (at 0 4) (layer F.Fab)
-      (effects (font (size 1 1) (thickness 0.15)))
-    )
-    (fp_circle (center 0 0) (end 3.25 0) (layer F.CrtYd) (width 0.05))
-    (fp_circle (center 0 0) (end 3 0) (layer Cmts.User) (width 0.15))
-    (fp_text user %R (at 0.3 0) (layer F.Fab)
-      (effects (font (size 1 1) (thickness 0.15)))
-    )
-    (pad 1 np_thru_hole circle (at 0 0) (size 3 3) (drill 3) (layers *.Cu *.Mask))
-  )
-  (module MountingHole:MountingHole_3mm (layer F.Cu)
-    (at 186.37 64.45)
-    (descr "Mounting Hole 3mm, no annular")
-    (tags "mounting hole 3mm no annular")
-    (attr virtual)
-    (fp_text reference HE16 (at 0 -4) (layer F.SilkS) hide
-      (effects (font (size 1 1) (thickness 0.15)))
-    )

Commit message: edge cuts adjusted
Parts:
- removed HA0, HA17, HB0, HB17, HJ0, HJ17, HK0, HK17: MountingHole, MountingHole:MountingHole_3mm
- moved J1 44.9 mm to (39.0, 100.0)
- moved J0 44.0 mm to (39.0, 49.2)
- moved J3 35.4 mm to (181.3, 100.0)
- moved J2 32.0 mm to (181.3, 49.2)
Other:
- outline, holes or cut-outs redrawn
Changed lines of the file:
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@@
   (general
     (thickness 1.6)
-    (drawings 4)
+    (drawings 12)
     (tracks 0)
     (zones 0)
-    (modules 211)
+    (modules 203)
     (nets 2)
   )
@@
   )
   (module Connector_Wire:SolderWirePad_1x01_Drill1mm (layer F.Cu)
-    (at 212.5472 83.4644)
+    (at 181.29 100.01)
     (descr "Wire solder connection")
     (tags connector)
@@
   )
   (module Connector_Wire:SolderWirePad_1x01_Drill1mm (layer F.Cu)
-    (at 212.5472 55.9054)
+    (at 181.29 49.21)
     (descr "Wire solder connection")
     (tags connector)
@@
   )
   (module Connector_Wire:SolderWirePad_1x01_Drill1mm (layer F.Cu)
-    (at -3.81 86.5378)
+    (at 39.05 100.01)
     (descr "Wire solder connection")
     (tags connector)
@@
   )
   (module Connector_Wire:SolderWirePad_1x01_Drill1mm (layer F.Cu)
-    (at -3.7338 59.69)
+    (at 39.05 49.21)
     (descr "Wire solder connection")
     (tags connector)
@@
   )
   (module MountingHole:MountingHole_3mm (layer F.Cu)
-    (at 196.53 125.41)
-    (descr "Mounting Hole 3mm, no annular")
-    (tags "mounting hole 3mm no annular")
-    (attr virtual)
-    (fp_text reference HK17 (at 0 -4) (layer F.SilkS) hide
-      (effects (font (size 1 1) (thickness 0.15)))
-    )
-    (fp_text value MountingHole (at 0 4) (layer F.Fab)
-      (effects (font (size 1 1) (thickness 0.15)))
-    )
-    (fp_circle (center 0 0) (end 3.25 0) (layer F.CrtYd) (width 0.05))
-    (fp_circle (center 0 0) (end 3 0) (layer Cmts.User) (width 0.15))
-    (fp_text user %R (at 0.3 0) (layer F.Fab)
-      (effects (font (size 1 1) (thickness 0.15)))
-    )
-    (pad 1 np_thru_hole circle (at 0 0) (size 3 3) (drill 3) (layers *.Cu *.Mask))
-  )
-  (module MountingHole:MountingHole_3mm (layer F.Cu)
     (at 186.37 125.41)
     (descr "Mounting Hole 3mm, no annular")
@@
   )
   (module MountingHole:MountingHole_3mm (layer F.Cu)
-    (at 23.81 125.41)
-    (descr "Mounting Hole 3mm, no annular")
-    (tags "mounting hole 3mm no annular")
-    (attr virtual)
-    (fp_text reference HK0 (at 0 -4) (layer F.SilkS) hide
-      (effects (font (size 1 1) (thickness 0.15)))
-    )
-    (fp_text value MountingHole (at 0 4) (layer F.Fab)
-      (effects (font (size 1 1) (thickness 0.15)))
-    )
-    (fp_circle (center 0 0) (end 3.25 0) (layer F.CrtYd) (width 0.05))
-    (fp_circle (center 0 0) (end 3 0) (layer Cmts.User) (width 0.15))
-    (fp_text user %R (at 0.3 0) (layer F.Fab)
-      (effects (font (size 1 1) (thickness 0.15)))
-    )
-    (pad 1 np_thru_hole circle (at 0 0) (size 3 3) (drill 3) (layers *.Cu *.Mask))
-  )
-  (module MountingHole:MountingHole_3mm (layer F.Cu)
-    (at 196.53 115.25)
-    (descr "Mounting Hole 3mm, no annular")
-    (tags "mounting hole 3mm no annular")
-    (attr virtual)
-    (fp_text reference HJ17 (at 0 -4) (layer F.SilkS) hide
-      (effects (font (size 1 1) (thickness 0.15)))
-    )
-    (fp_text value MountingHole (at 0 4) (layer F.Fab)
-      (effects (font (size 1 1) (thickness 0.15)))
-    )
-    (fp_circle (center 0 0) (end 3.25 0) (layer F.CrtYd) (width 0.05))
-    (fp_circle (center 0 0) (end 3 0) (layer Cmts.User) (width 0.15))
-    (fp_text user %R (at 0.3 0) (layer F.Fab)
-      (effects (font (size 1 1) (thickness 0.15)))
-    )
-    (pad 1 np_thru_hole circle (at 0 0) (size 3 3) (drill 3) (layers *.Cu *.Mask))
-  )
-  (module MountingHole:MountingHole_3mm (layer F.Cu)
     (at 186.37 115.25)
     (descr "Mounting Hole 3mm, no annular")
@@
   )
   (module MountingHole:MountingHole_3mm (layer F.Cu)
-    (at 23.81 115.25)
-    (descr "Mounting Hole 3mm, no annular")
-    (tags "mounting hole 3mm no annular")
-    (attr virtual)
-    (fp_text reference HJ0 (at 0 -4) (layer F.SilkS) hide
-      (effects (font (size 1 1) (thickness 0.15)))
-    )
-    (fp_text value MountingHole (at 0 4) (layer F.Fab)
-      (effects (font (size 1 1) (thickness 0.15)))
-    )
-    (fp_circle (center 0 0) (end 3.25 0) (layer F.CrtYd) (width 0.05))
-    (fp_circle (center 0 0) (end 3 0) (layer Cmts.User) (width 0.15))
-    (fp_text user %R (at 0.3 0) (layer F.Fab)
-      (effects (font (size 1 1) (thickness 0.15)))
-    )
-    (pad 1 np_thru_hole circle (at 0 0) (size 3 3) (drill 3) (layers *.Cu *.Mask))
-  )
-  (module MountingHole:MountingHole_3mm (layer F.Cu)
     (at 196.53 105.09)
     (descr "Mounting Hole 3mm, no annular")
@@
   )
   (module MountingHole:MountingHole_3mm (layer F.Cu)
-    (at 196.53 33.97)
-    (descr "Mounting Hole 3mm, no annular")
-    (tags "mounting hole 3mm no annular")
-    (attr virtual)
-    (fp_text reference HB17 (at 0 -4) (layer F.SilkS) hide
-      (effects (font (size 1 1) (thickness 0.15)))
-    )
-    (fp_text value MountingHole (at 0 4) (layer F.Fab)
-      (effects (font (size 1 1) (thickness 0.15)))
-    )
-    (fp_circle (center 0 0) (end 3.25 0) (layer F.CrtYd) (width 0.05))
-    (fp_circle (center 0 0) (end 3 0) (layer Cmts.User) (width 0.15))
-    (fp_text user %R (at 0.3 0) (layer F.Fab)
-      (effects (font (size 1 1) (thickness 0.15)))
-    )
-    (pad 1 np_thru_hole circle (at 0 0) (size 3 3) (drill 3) (layers *.Cu *.Mask))
-  )
-  (module MountingHole:MountingHole_3mm (layer F.Cu)
     (at 186.37 33.97)
     (descr "Mounting Hole 3mm, no annular")
@@
   )
   (module MountingHole:MountingHole_3mm (layer F.Cu)
-    (at 23.81 33.97)
-    (descr "Mounting Hole 3mm, no annular")
-    (tags "mounting hole 3mm no annular")
-    (attr virtual)
-    (fp_text reference HB0 (at 0 -4) (layer F.SilkS) hide
-      (effects (font (size 1 1) (thickness 0.15)))
-    )
-    (fp_text value MountingHole (at 0 4) (layer F.Fab)
-      (effects (font (size 1 1) (thickness 0.15)))
-    )
-    (fp_circle (center 0 0) (end 3.25 0) (layer F.CrtYd) (width 0.05))
-    (fp_circle (center 0 0) (end 3 0) (layer Cmts.User) (width 0.15))
-    (fp_text user %R (at 0.3 0) (layer F.Fab)
-      (effects (font (size 1 1) (thickness 0.15)))
-    )
-    (pad 1 np_thru_hole circle (at 0 0) (size 3 3) (drill 3) (layers *.Cu *.Mask))
-  )
-  (module MountingHole:MountingHole_3mm (layer F.Cu)
-    (at 196.53 23.81)
-    (descr "Mounting Hole 3mm, no annular")
-    (tags "mounting hole 3mm no annular")
-    (attr virtual)
-    (fp_text reference HA17 (at 0 -4) (layer F.SilkS) hide
-      (effects (font (size 1 1) (thickness 0.15)))
-    )
-    (fp_text value MountingHole (at 0 4) (layer F.Fab)
-      (effects (font (size 1 1) (thickness 0.15)))
-    )
-    (fp_circle (center 0 0) (end 3.25 0) (layer F.CrtYd) (width 0.05))
-    (fp_circle (center 0 0) (end 3 0) (layer Cmts.User) (width 0.15))
-    (fp_text user %R (at 0.3 0) (layer F.Fab)
-      (effects (font (size 1 1) (thickness 0.15)))
-    )
-    (pad 1 np_thru_hole circle (at 0 0) (size 3 3) (drill 3) (layers *.Cu *.Mask))
-  )
-  (module MountingHole:MountingHole_3mm (layer F.Cu)
     (at 186.37 23.81)
     (descr "Mounting Hole 3mm, no annular")
@@
     (pad 1 np_thru_hole circle (at 0 0) (size 3 3) (drill 3) (layers *.Cu *.Mask))
   )
-  (module MountingHole:MountingHole_3mm (layer F.Cu)
-    (at 23.81 23.81)
-    (descr "Mounting Hole 3mm, no annular")
-    (tags "mounting hole 3mm no annular")
-    (attr virtual)
-    (fp_text reference HA0 (at 0 -4) (layer F.SilkS) hide
-      (effects (font (size 1 1) (thickness 0.15)))
-    )
-    (fp_text value MountingHole (at 0 4) (layer F.Fab)
-      (effects (font (size 1 1) (thickness 0.15)))
-    )
-    (fp_circle (center 0 0) (end 3.25 0) (layer F.CrtYd) (width 0.05))
-    (fp_circle (center 0 0) (end 3 0) (layer Cmts.User) (width 0.15))
-    (fp_text user %R (at 0.3 0) (layer F.Fab)
-      (effects (font (size 1 1) (thickness 0.15)))
-    )
-    (pad 1 np_thru_hole circle (at 0 0) (size 3 3) (drill 3) (layers *.Cu *.Mask))
-  )
-  (gr_line (start 18.67 129.61) (end 201.67 129.61) (layer Edge.Cuts) (width 0.05))
-  (gr_line (start 201.67 19.61) (end 201.67 129.61) (layer Edge.Cuts) (width 0.05))
-  (gr_line (start 18.67 19.61) (end 201.67 19.61) (layer Edge.Cuts) (width 0.05))
-  (gr_line (start 18.67 19.61) (end 18.67 129.61) (layer Edge.Cuts) (width 0.05))
+  (gr_line (start 194.67 110.61) (end 194.67 129.61) (layer Edge.Cuts) (width 0.05))
+  (gr_line (start 194.67 110.61) (end 201.67 110.61) (layer Edge.Cuts) (width 0.05))
+  (gr_line (start 194.67 38.61) (end 201.67 38.61) (layer Edge.Cuts) (width 0.05))
+  (gr_line (start 194.67 19.61) (end 194.67 38.61) (layer Edge.Cuts) (width 0.05))
+  (gr_line (start 25.67 110.61) (end 25.67 129.61) (layer Edge.Cuts) (width 0.05))
+  (gr_line (start 18.67 110.61) (end 25.67 110.61) (layer Edge.Cuts) (width 0.05))
+  (gr_line (start 25.67 19.61) (end 25.67 38.61) (layer Edge.Cuts) (width 0.05))
+  (gr_line (start 18.67 38.61) (end 25.67 38.61) (layer Edge.Cuts) (width 0.05))
+  (gr_line (start 25.67 129.61) (end 194.67 129.61) (layer Edge.Cuts) (width 0.05))
+  (gr_line (start 201.67 38.61) (end 201.67 110.61) (layer Edge.Cuts) (width 0.05))
+  (gr_line (start 25.67 19.61) (end 194.67 19.61) (layer Edge.Cuts) (width 0.05))
+  (gr_line (start 18.67 38.61) (end 18.67 110.61) (layer Edge.Cuts) (width 0.05))
 )
