File: A_BACKPLATES/A03/A03.kicad_pcb (KiCad board)
At the start: 2 copper layers, 65 x 30 mm, 74 parts, among them J0 Conn_01x01_Male, J1 Conn_01x01_Male, J2 Conn_01x01_Male, J3 Conn_01x01_Male

Commit message: A03 finished
Parts:
- removed HA0, HA10, HA11, HA12, HA13, HA14, HA15, HA16, HA17, HA6, HA7, HA8, HA9, HB0, HB10, HB11, HB12, HB13, HB14, HB15, HB16, HB17, HB6, HB7, HB8, HB9, HC0, HC10, HC11, HC12, HC13, HC14, HC15, HC16, HC17, HC6, HC7, HC8, HC9, HZ10, HZ11, HZ12, HZ13, HZ14, HZ15, HZ4, HZ5, HZ6, HZ7, HZ8, HZ9: MountingHole, MountingHole:MountingHole_3mm
- removed J2, J3: Conn_01x01_Male, Connector_Wire:SolderWirePad_1x01_Drill1mm
- added REF**: OSHW-Symbol_6.7x6mm_Copper, Symbol:OSHW-Symbol_6.7x6mm_Copper, B.Cu at (69.4, 39.0)
- added REF**: OSHW-Symbol_6.7x6mm_SilkScreen, Symbol:OSHW-Symbol_6.7x6mm_SilkScreen, F.Cu at (38.2, 28.7)
- added REF**: OSHW-Symbol_6.7x6mm_SilkScreen, Symbol:OSHW-Symbol_6.7x6mm_SilkScreen, B.Cu at (38.7, 39.4)
- added REF**: OSHW-Symbol_6.7x6mm_Copper, Symbol:OSHW-Symbol_6.7x6mm_Copper, F.Cu at (69.3, 28.7)
- moved J0 206.5 mm to (28.9, 34.0), turned to 270 degrees
- moved HZ1 202.9 mm to (25.3, 45.5)
- moved HZ0 191.6 mm to (25.3, 22.5)
- moved HZ3 165.5 mm to (83.3, 45.5)
- moved J1 154.9 mm to (79.7, 34.0)
- moved HZ2 153.9 mm to (83.3, 22.5)
Routing:
- added copper zone on B.Cu, net Net-(J0-Pad1)
- added copper zone on F.Cu, net Net-(J0-Pad1)
Other:
- board text added: "A03_BACKPLATE"
