File: A_BACKPLATES/A05/A05.kicad_pcb (KiCad board)
At the start: 2 copper layers, 88.9 x 68.6 mm, 72 parts, among them J0 Conn_01x01_Male, J1 Conn_01x01_Male, J2 Conn_01x01_Male, J3 Conn_01x01_Male

Commit message: fixed misplaced mounting hole
Parts:
- removed HB0, HB7, HB8, HF0, HF7: MountingHole, MountingHole:MountingHole_3mm
- moved J2 10.2 mm to (79.7, 28.9)
- moved J3 10.2 mm to (79.7, 79.7)
- moved HZ1 3.00 mm to (94.0, 78.3)
- moved HZ2 3.00 mm to (25.9, 78.3)
Routing:
- added copper zone on F.Cu, net Net-(J0-Pad1)
Changed lines of the file:
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@@
     (tracks 0)
     (zones 0)
-    (modules 72)
+    (modules 67)
     (nets 2)
   )
@@
     (visible_elements FFFFFF7F)
     (pcbplotparams
-      (layerselection 0x010fc_ffffffff)
+      (layerselection 0x01000_7fffffff)
       (usegerberextensions false)
       (usegerberattributes false)
@@
       (padsonsilk false)
       (subtractmaskfromsilk false)
-      (outputformat 1)
+      (outputformat 5)
       (mirror false)
-      (drillshape 1)
+      (drillshape 2)
       (scaleselection 1)
-      (outputdirectory ""))
+      (outputdirectory "./"))
   )
   (net 0 "")
@@
   )
   (module MountingHole:MountingHole_4mm (layer F.Cu)
-    (at 25.95 75.29)
+    (at 25.95 78.29)
     (descr "Mounting Hole 4mm, no annular")
     (tags "mounting hole 4mm no annular")
@@
   )
   (module MountingHole:MountingHole_4mm (layer F.Cu)
-    (at 93.95 75.29)
+    (at 93.95 78.29)
     (descr "Mounting Hole 4mm, no annular")
     (tags "mounting hole 4mm no annular")
@@
   )
   (module Connector_Wire:SolderWirePad_1x01_Drill1mm (layer F.Cu)
-    (at 89.85 79.69)
+    (at 79.69 79.69)
     (descr "Wire solder connection")
     (tags connector)
@@
   )
   (module Connector_Wire:SolderWirePad_1x01_Drill1mm (layer F.Cu)
-    (at 89.85 28.89)
+    (at 79.69 28.89)
     (descr "Wire solder connection")
     (tags connector)
@@
   )
   (module MountingHole:MountingHole_3mm (layer F.Cu)
-    (at 94.93 74.61)
-    (descr "Mounting Hole 3mm, no annular")
-    (tags "mounting hole 3mm no annular")
-    (attr virtual)
-    (fp_text reference HF7 (at 0 -4) (layer F.SilkS) hide
-      (effects (font (size 1 1) (thickness 0.15)))
-    )
-    (fp_text value MountingHole (at 0 4) (layer F.Fab)
-      (effects (font (size 1 1) (thickness 0.15)))
-    )
-    (fp_circle (center 0 0) (end 3.25 0) (layer F.CrtYd) (width 0.05))
-    (fp_circle (center 0 0) (end 3 0) (layer Cmts.User) (width 0.15))
-    (fp_text user %R (at 0.3 0) (layer F.Fab)
-      (effects (font (size 1 1) (thickness 0.15)))
-    )
-    (pad 1 np_thru_hole circle (at 0 0) (size 3 3) (drill 3) (layers *.Cu *.Mask))
-  )
-  (module MountingHole:MountingHole_3mm (layer F.Cu)
     (at 84.77 74.61)
     (descr "Mounting Hole 3mm, no annular")
@@
   )
   (module MountingHole:MountingHole_3mm (layer F.Cu)
-    (at 23.81 74.61)
-    (descr "Mounting Hole 3mm, no annular")
-    (tags "mounting hole 3mm no annular")
-    (attr virtual)
-    (fp_text reference HF0 (at 0 -4) (layer F.SilkS) hide
-      (effects (font (size 1 1) (thickness 0.15)))
-    )
-    (fp_text value MountingHole (at 0 4) (layer F.Fab)
-      (effects (font (size 1 1) (thickness 0.15)))
-    )
-    (fp_circle (center 0 0) (end 3.25 0) (layer F.CrtYd) (width 0.05))
-    (fp_circle (center 0 0) (end 3 0) (layer Cmts.User) (width 0.15))
-    (fp_text user %R (at 0.3 0) (layer F.Fab)
-      (effects (font (size 1 1) (thickness 0.15)))
-    )
-    (pad 1 np_thru_hole circle (at 0 0) (size 3 3) (drill 3) (layers *.Cu *.Mask))
-  )
-  (module MountingHole:MountingHole_3mm (layer F.Cu)
     (at 105.09 64.45)
     (descr "Mounting Hole 3mm, no annular")
@@
   )
   (module MountingHole:MountingHole_3mm (layer F.Cu)
-    (at 105.09 33.97)
-    (descr "Mounting Hole 3mm, no annular")
-    (tags "mounting hole 3mm no annular")
-    (attr virtual)
-    (fp_text reference HB8 (at 0 -4) (layer F.SilkS) hide
-      (effects (font (size 1 1) (thickness 0.15)))
-    )
-    (fp_text value MountingHole (at 0 4) (layer F.Fab)
-      (effects (font (size 1 1) (thickness 0.15)))
-    )
-    (fp_circle (center 0 0) (end 3.25 0) (layer F.CrtYd) (width 0.05))
-    (fp_circle (center 0 0) (end 3 0) (layer Cmts.User) (width 0.15))
-    (fp_text user %R (at 0.3 0) (layer F.Fab)
-      (effects (font (size 1 1) (thickness 0.15)))
-    )
-    (pad 1 np_thru_hole circle (at 0 0) (size 3 3) (drill 3) (layers *.Cu *.Mask))
-  )
-  (module MountingHole:MountingHole_3mm (layer F.Cu)
-    (at 94.93 33.97)
-    (descr "Mounting Hole 3mm, no annular")
-    (tags "mounting hole 3mm no annular")
-    (attr virtual)
-    (fp_text reference HB7 (at 0 -4) (layer F.SilkS) hide
-      (effects (font (size 1 1) (thickness 0.15)))
-    )
-    (fp_text value MountingHole (at 0 4) (layer F.Fab)
-      (effects (font (size 1 1) (thickness 0.15)))
-    )
-    (fp_circle (center 0 0) (end 3.25 0) (layer F.CrtYd) (width 0.05))
-    (fp_circle (center 0 0) (end 3 0) (layer Cmts.User) (width 0.15))
-    (fp_text user %R (at 0.3 0) (layer F.Fab)
-      (effects (font (size 1 1) (thickness 0.15)))
-    )
-    (pad 1 np_thru_hole circle (at 0 0) (size 3 3) (drill 3) (layers *.Cu *.Mask))
-  )
-  (module MountingHole:MountingHole_3mm (layer F.Cu)
     (at 84.77 33.97)
     (descr "Mounting Hole 3mm, no annular")
@@
     (attr virtual)
     (fp_text reference HB1 (at 0 -4) (layer F.SilkS) hide
-      (effects (font (size 1 1) (thickness 0.15)))
-    )
-    (fp_text value MountingHole (at 0 4) (layer F.Fab)
-      (effects (font (size 1 1) (thickness 0.15)))
-    )
-    (fp_circle (center 0 0) (end 3.25 0) (layer F.CrtYd) (width 0.05))
-    (fp_circle (center 0 0) (end 3 0) (layer Cmts.User) (width 0.15))
-    (fp_text user %R (at 0.3 0) (layer F.Fab)
-      (effects (font (size 1 1) (thickness 0.15)))
-    )
-    (pad 1 np_thru_hole circle (at 0 0) (size 3 3) (drill 3) (layers *.Cu *.Mask))
-  )
-  (module MountingHole:MountingHole_3mm (layer F.Cu)
-    (at 23.81 33.97)
-    (descr "Mounting Hole 3mm, no annular")
-    (tags "mounting hole 3mm no annular")
-    (attr virtual)
-    (fp_text reference HB0 (at 0 -4) (layer F.SilkS) hide
       (effects (font (size 1 1) (thickness 0.15)))
     )
@@
   (gr_line (start 20 20) (end 108.9 20) (layer Edge.Cuts) (width 0.05))
   (gr_line (start 20 20) (end 20 88.58) (layer Edge.Cuts) (width 0.05))
+  (zone (net 1) (net_name "Net-(J0-Pad1)") (layer F.Cu) (hatch edge 0.508)
+    (connect_pads (clearance 0.508))
+    (min_thickness 0.254)
+    (fill yes (arc_segments 32) (thermal_gap 0.508) (thermal_bridge_width 0.508))
+    (polygon
+      (pts
+        (xy 108.3564 88.138) (xy 20.3708 88.138) (xy 20.4724 20.447) (xy 108.3564 20.4724)
+      )
+    )
+  )
 )

Commit message: A05 gerber files
Parts:
- added REF**: OSHW-Symbol_6.7x6mm_Copper, Symbol:OSHW-Symbol_6.7x6mm_Copper, B.Cu at (79.6, 49.3)
- added REF**: OSHW-Symbol_6.7x6mm_Copper, Symbol:OSHW-Symbol_6.7x6mm_Copper, F.Cu at (79.6, 59.1)
- added REF**: OSHW-Symbol_6.7x6mm_SilkScreen, Symbol:OSHW-Symbol_6.7x6mm_SilkScreen, F.Cu at (38.6, 58.9)
- added REF**: OSHW-Symbol_6.7x6mm_SilkScreen, Symbol:OSHW-Symbol_6.7x6mm_SilkScreen, B.Cu at (38.8, 49.3)
Routing:
- added copper zone on B.Cu, net Net-(J0-Pad1)
Other:
- board text added: "A05_BACKPLATE"
