File: B_SCREW_TERMINAL_WIRE_CONNECTORS/B01/B01.kicad_pcb (KiCad board)
At the start: 2 copper layers, 27.9 x 17.8 mm, 8 parts, among them J0 Conn_01x01_Male, J1 Conn_01x01_Male, J4 Conn_01x04_Female, J5 Conn_01x04_Female

Commit message: B00 gerbers single
Parts:
- added REF**: OSHW-Symbol_6.7x6mm_SilkScreen, Symbol:OSHW-Symbol_6.7x6mm_SilkScreen, B.Cu at (40.1, 28.9)
- added REF**: OSHW-Symbol_6.7x6mm_SilkScreen, Symbol:OSHW-Symbol_6.7x6mm_SilkScreen, F.Cu at (27.6, 28.8)
- moved J0 46.2 mm to (23.8, 28.9)
- moved J1 25.7 mm to (44.1, 28.9)
Routing:
- net Net-(J4-Pad4): track 0.00 -> 19.0 mm
- net Net-(J4-Pad3): track 0.00 -> 19.0 mm
- net Net-(J4-Pad2): track 0.00 -> 19.0 mm
- net Net-(J4-Pad1): track 0.00 -> 19.0 mm
- added copper zone on B.Cu, net Net-(J0-Pad1)
- added copper zone on F.Cu, net Net-(J0-Pad1)
Other:
- net class Default: trace_width 0.25 -> 0.75
- board text added: "B01_S2S"
