File: B_SCREW_TERMINAL_WIRE_CONNECTORS/B02/B02.kicad_pcb (KiCad board)
At the start: 2 copper layers, 38.1 x 17.8 mm, 8 parts, among them J0 Conn_01x01_Male, J1 Conn_01x01_Male, J4 Conn_01x07_Female, J5 Conn_01x07_Female

Commit message: B02 gerber single an panel
Parts:
- added REF**: OSHW-Symbol_6.7x6mm_SilkScreen, Symbol:OSHW-Symbol_6.7x6mm_SilkScreen, B.Cu at (50.4, 29.0)
- added REF**: OSHW-Symbol_6.7x6mm_SilkScreen, Symbol:OSHW-Symbol_6.7x6mm_SilkScreen, F.Cu at (27.7, 28.8)
Routing:
- net Net-(J4-Pad7): track 0.00 -> 18.5 mm
- net Net-(J4-Pad6): track 0.00 -> 18.5 mm
- net Net-(J4-Pad5): track 0.00 -> 18.5 mm
- net Net-(J4-Pad4): track 0.00 -> 18.5 mm
- net Net-(J4-Pad3): track 0.00 -> 18.5 mm
- net Net-(J4-Pad2): track 0.00 -> 18.5 mm
- net Net-(J4-Pad1): track 0.00 -> 18.5 mm
- added copper zone on B.Cu, net Net-(J0-Pad1)
- added copper zone on F.Cu, net Net-(J0-Pad1)
Other:
- net class Default: trace_width 0.25 -> 0.75
- board text added: "B02_S2S"
