File: B_SCREW_TERMINAL_WIRE_CONNECTORS/B03/B03.kicad_pcb (KiCad board)
At the start: 2 copper layers, 48.3 x 17.8 mm, 8 parts, among them J0 Conn_01x01_Male, J1 Conn_01x01_Male, J2 Conn_01x10_Female, J3 Conn_01x10_Female

Commit message: B03 single gerbers
Parts:
- added REF**: OSHW-Symbol_6.7x6mm_SilkScreen, Symbol:OSHW-Symbol_6.7x6mm_SilkScreen, B.Cu at (60.7, 29.0)
- added REF**: OSHW-Symbol_6.7x6mm_SilkScreen, Symbol:OSHW-Symbol_6.7x6mm_SilkScreen, F.Cu at (27.7, 28.8)
Routing:
- added copper zone on B.Cu, net Net-(J0-Pad1)
- added copper zone on F.Cu, net Net-(J0-Pad1)
Other:
- board text added: "B03_S2S"
