File: D_ELECTRONICS/D00/D00.kicad_pcb (KiCad board)
At the start: 2 copper layers, 58.4 x 27.9 mm, 15 parts, among them J0 Conn_01x01_Male, J1 Conn_01x01_Male, J2 Conn_01x01_Male, J3 Conn_01x01_Male, J4 Conn_01x02_Female, J5 Conn_01x04_Female

Commit message: silkscreen polarity fixed, added B cu traces
Routing:
- net Net-(J4-Pad2): track 10.6 -> 21.2 mm
- net Net-(J4-Pad1): track 10.6 -> 21.2 mm
- net Net-(J5-Pad3): track 12.7 -> 16.2 mm
- net Net-(J5-Pad1): track 12.7 -> 16.2 mm
Other:
- board text added: "+ + - -"
- board text removed: "- - + +"
Changed lines of the file:
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@@
     (thickness 1.6)
     (drawings 9)
-    (tracks 10)
+    (tracks 16)
     (zones 0)
     (modules 15)
@@
     (pad 1 np_thru_hole circle (at 0 0) (size 3 3) (drill 3) (layers *.Cu *.Mask))
   )
-  (gr_text "- -  + +" (at 74.8538 33.9852 90) (layer F.SilkS)
+  (gr_text "+ +  - -" (at 74.8538 33.9852 90) (layer F.SilkS)
     (effects (font (size 1.5 1.5) (thickness 0.15)))
   )
@@
   (segment (start 24.9816 36.47) (end 24.2316 35.72) (width 0.75) (layer F.Cu) (net 2))
   (segment (start 34.51 36.47) (end 24.9816 36.47) (width 0.75) (layer F.Cu) (net 2))
+  (segment (start 24.9816 36.47) (end 24.2316 35.72) (width 0.75) (layer B.Cu) (net 2))
+  (segment (start 34.51 36.47) (end 24.9816 36.47) (width 0.75) (layer B.Cu) (net 2))
   (segment (start 24.9816 31.47) (end 24.2316 32.22) (width 0.75) (layer F.Cu) (net 3))
   (segment (start 34.51 31.47) (end 24.9816 31.47) (width 0.75) (layer F.Cu) (net 3))
+  (segment (start 24.9816 31.47) (end 24.2316 32.22) (width 0.75) (layer B.Cu) (net 3))
+  (segment (start 34.51 31.47) (end 24.9816 31.47) (width 0.75) (layer B.Cu) (net 3))
   (segment (start 66.36 28.72) (end 72.0852 28.72) (width 0.75) (layer F.Cu) (net 4))
   (segment (start 63.91 26.27) (end 66.36 28.72) (width 0.75) (layer F.Cu) (net 4))
   (segment (start 72.0852 28.72) (end 72.0852 32.22) (width 0.75) (layer F.Cu) (net 4))
+  (segment (start 72.0852 28.72) (end 72.0852 32.22) (width 0.75) (layer B.Cu) (net 4))
   (segment (start 66.36 39.22) (end 63.91 41.67) (width 0.75) (layer F.Cu) (net 5))
   (segment (start 72.0852 39.22) (end 66.36 39.22) (width 0.75) (layer F.Cu) (net 5))
   (segment (start 72.0852 35.72) (end 72.0852 39.22) (width 0.75) (layer F.Cu) (net 5))
+  (segment (start 72.0852 35.72) (end 72.0852 39.22) (width 0.75) (layer B.Cu) (net 5))
   (zone (net 1) (net_name "Net-(J0-Pad1)") (layer F.Cu) (hatch edge 0.508)
     (connect_pads (clearance 0.508))
