File: D_ELECTRONICS/D00/D00.sch (KiCad schematic (older format))
At the start: 11 parts, among them J0 Conn_01x01_Male, J1 Conn_01x01_Male, J2 Conn_01x01_Male, J3 Conn_01x01_Male, J4 Conn_01x02_Female, J5 Conn_01x04_Female

Commit message: bigger screw terminal for the AC side
Parts:
- J4: footprint TerminalBlock_4Ucon:TerminalBlock_4Ucon_1x02_P3.50mm_Horizontal -> TerminalBlock_RND:TerminalBlock_RND_205-00001_1x02_P5.00mm_Horizontal
Changed lines of the file:
@@
 F 0 "J4" H 5542 2735 50  0000 C CNN
 F 1 "Conn_01x02_Female" H 5542 2644 50  0000 C CNN
-F 2 "TerminalBlock_4Ucon:TerminalBlock_4Ucon_1x02_P3.50mm_Horizontal" H 5650 2550 50  0001 C CNN
+F 2 "TerminalBlock_RND:TerminalBlock_RND_205-00001_1x02_P5.00mm_Horizontal" H 5650 2550 50  0001 C CNN
 F 3 "~" H 5650 2550 50  0001 C CNN
 	1    5650 2550
