File: D_ELECTRONICS/D02/D02.sch (KiCad schematic (older format))
At the start: 19 parts, among them J0 Conn_01x01_Male, J1 Conn_01x01_Male, J2 Conn_01x01_Male, J3 Conn_01x01_Male, J4 USB_B_Micro, J5 Conn_01x02_Female, J6 Conn_01x03_Female, U1 AMS1117-3.3

Commit message: single panel
Parts:
- removed J2, J3: Conn_01x01_Male, Connector_Wire:SolderWirePad_1x01_Drill1mm, symbol Connector:Conn_01x01_Male
Connections:
- net at C1.2, C2.2, C3.2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: now also R1.2; no longer D1.1 (K)
- net at C3.1, C4.1, J6.2 (Pin_2)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: now also D1.2 (A); no longer R1.1
- new net: D1.1 (K), R1.1
Other:
- moved on the sheet: D1, R1
Changed lines of the file:
@@
-	1    0    0    -1
-$EndComp
-$Comp
-L Connector:Conn_01x01_Male J1
-U 1 1 5F5DB1C6
-P 6300 1000
-F 0 "J1" H 6408 1181 50  0000 C CNN
-F 1 "Conn_01x01_Male" H 6408 1090 50  0000 C CNN
-F 2 "Connector_Wire:SolderWirePad_1x01_Drill1mm" H 6300 1000 50  0001 C CNN
-F 3 "~" H 6300 1000 50  0001 C CNN
-	1    6300 1000
-	1    0    0    -1
-$EndComp
-$Comp
-L Connector:Conn_01x01_Male J2
-U 1 1 5F5DCAC3
-P 6300 1150
-F 0 "J2" H 6408 1331 50  0000 C CNN
-F 1 "Conn_01x01_Male" H 6408 1240 50  0000 C CNN
-F 2 "Connector_Wire:SolderWirePad_1x01_Drill1mm" H 6300 1150 50  0001 C CNN
-F 3 "~" H 6300 1150 50  0001 C CNN
-	1    6300 1150
-	1    0    0    -1
-$EndComp
-$Comp
-L Connector:Conn_01x01_Male J3
-U 1 1 5F5DDB13
-P 6300 1300
-F 0 "J3" H 6408 1481 50  0000 C CNN
-F 1 "Conn_01x01_Male" H 6408 1390 50  0000 C CNN
-F 2 "Connector_Wire:SolderWirePad_1x01_Drill1mm" H 6300 1300 50  0001 C CNN
-F 3 "~" H 6300 1300 50  0001 C CNN
-	1    6300 1300
 	1    0    0    -1
 $EndComp
@@
 Wire Wire Line
 	6750 1000 6500 1000
-Wire Wire Line
-	6500 1150 6750 1150
-Wire Wire Line
-	6750 1150 6750 1000
-Connection ~ 6750 1000
-Wire Wire Line
-	6500 1300 6750 1300
-Wire Wire Line
-	6750 1300 6750 1150
-Connection ~ 6750 1150
 Text Label 6250 1650 0    50   ~ 0
 GROUND_PLANE
@@
 Connection ~ 7450 3100
 Connection ~ 7700 2250
-Wire Wire Line
-	8200 2250 8000 2250
 Connection ~ 7700 3100
 Wire Wire Line
@@
 L Device:R R1
 U 1 1 5F6D8881
+P 8000 2900
+F 0 "R1" H 8070 2946 50  0000 L CNN
+F 1 "R" H 8070 2855 50  0000 L CNN
+F 2 "Resistor_THT:R_Axial_DIN0204_L3.6mm_D1.6mm_P2.54mm_Vertical" V 7930 2900 50  0001 C CNN
+F 3 "~" H 8000 2900 50  0001 C CNN
+	1    8000 2900
+	1    0    0    -1
+$EndComp
+$Comp
+L Device:LED D1
+U 1 1 5F6D9335
 P 8000 2450
-F 0 "R1" H 8070 2496 50  0000 L CNN
-F 1 "R" H 8070 2405 50  0000 L CNN
-F 2 "Resistor_THT:R_Axial_DIN0204_L3.6mm_D1.6mm_P2.54mm_Vertical" V 7930 2450 50  0001 C CNN
+F 0 "D1" V 8039 2333 50  0000 R CNN
+F 1 "LED" V 7948 2333 50  0000 R CNN
+F 2 "LED_THT:LED_D3.0mm" H 8000 2450 50  0001 C CNN
 F 3 "~" H 8000 2450 50  0001 C CNN
 	1    8000 2450
-	1    0    0    -1
-$EndComp
-$Comp
-L Device:LED D1
-U 1 1 5F6D9335
-P 8000 2850
-F 0 "D1" V 8039 2733 50  0000 R CNN
-F 1 "LED" V 7948 2733 50  0000 R CNN
-F 2 "LED_THT:LED_D3.0mm" H 8000 2850 50  0001 C CNN
-F 3 "~" H 8000 2850 50  0001 C CNN
-	1    8000 2850
 	0    -1   -1   0
 $EndComp
@@
 	5700 3100 6100 3100
 Wire Wire Line
-	8000 2700 8000 2600
-Wire Wire Line
-	8000 2300 8000 2250
-Connection ~ 8000 2250
-Wire Wire Line
-	8000 2250 7700 2250
-Wire Wire Line
-	8000 3000 8000 3100
-Wire Wire Line
-	7700 3100 8000 3100
-Wire Wire Line
 	8200 2350 8150 2350
 Wire Wire Line
 	8150 2350 8150 3100
-Wire Wire Line
-	8150 3100 8000 3100
-Connection ~ 8000 3100
 Wire Wire Line
 	5900 3450 6050 3450
@@
 	1    0    0    -1
 $EndComp
+Wire Wire Line
+	7700 2250 8000 2250
+Wire Wire Line
+	7700 3100 8000 3100
+Wire Wire Line
+	8000 2300 8000 2250
+Connection ~ 8000 2250
+Wire Wire Line
+	8000 2250 8200 2250
+Wire Wire Line
+	8000 2600 8000 2750
+Wire Wire Line
+	8000 3050 8000 3100
+Connection ~ 8000 3100
+Wire Wire Line
+	8000 3100 8150 3100
+$Comp
+L Connector:Conn_01x01_Male J1
+U 1 1 5F5DB1C6
+P 6300 1000
+F 0 "J1" H 6408 1181 50  0000 C CNN
+F 1 "Conn_01x01_Male" H 6408 1090 50  0000 C CNN
+F 2 "Connector_Wire:SolderWirePad_1x01_Drill1mm" H 6300 1000 50  0001 C CNN
+F 3 "~" H 6300 1000 50  0001 C CNN
+	1    6300 1000
+	1    0    0    -1
+$EndComp
