File: D_ELECTRONICS/D02/D02.kicad_pcb (KiCad board)
At the start: 2 copper layers, 59.8 x 17.8 mm, 19 parts, among them J0 Conn_01x01_Male, J1 Conn_01x01_Male, J2 Conn_01x01_Male, J3 Conn_01x01_Male, J4 USB_B_Micro, J5 Conn_01x02_Female, J6 Conn_01x03_Female, U1 AMS1117-3.3

Commit message: some traces routed
Parts:
- moved C1 0.84 mm to (46.9, 28.1)
- moved C4 0.26 mm to (46.9, 22.8)
- moved R1 0.10 mm to (41.2, 29.6)
Routing:
- net Net-(C1-Pad2): track 0.00 -> 43.7 mm, vias 0 -> 2
- net Net-(C1-Pad1): track 0.00 -> 28.2 mm
- net Net-(C3-Pad1): track 0.00 -> 15.7 mm
Other:
- net class Default: trace_width 0.25 -> 0.5
Changed lines of the file:
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@@
     (thickness 1.6)
     (drawings 4)
-    (tracks 0)
+    (tracks 51)
     (zones 0)
     (modules 19)
@@
   )
   (setup
-    (last_trace_width 0.25)
+    (last_trace_width 0.5)
     (trace_clearance 0.2)
     (zone_clearance 0.508)
@@
   (net_class Default "This is the default net class."
     (clearance 0.2)
-    (trace_width 0.25)
+    (trace_width 0.5)
     (via_dia 0.8)
     (via_drill 0.4)
@@
   )
   (module Resistor_THT:R_Axial_DIN0204_L3.6mm_D1.6mm_P2.54mm_Vertical (layer F.Cu)
-    (at 41.0718 29.5656 90)
+    (at 41.1734 29.5656 90)
     (descr "Resistor, Axial_DIN0204 series, Axial, Vertical, pin pitch=2.54mm, 0.167W, length*diameter=3.6*1.6mm^2, http://cdn-reichelt.de/documents/datenblatt/B400/1_4W%23YAG.pdf")
     (tags "Resistor Axial_DIN0204 series Axial Vertical pin pitch 2.54mm 0.167W length 3.6mm diameter 1.6mm")
@@
   )
   (module Capacitor_SMD:C_0805_2012Metric_Pad1.15x1.40mm_HandSolder (layer F.Cu)
-    (at 46.609 22.7838 90)
+    (at 46.863 22.8346 90)
     (descr "Capacitor SMD 0805 (2012 Metric), square (rectangular) end terminal, IPC_7351 nominal with elongated pad for handsoldering. (Body size source: https://docs.google.com/spreadsheets/d/1BsfQQcO9C6DZCsRaXUlFlo91Tg2WpOkGARC1WS5S8t0/edit?usp=sharing), generated with kicad-footprint-generator")
     (tags "capacitor handsolder")
@@
   )
   (module Capacitor_SMD:C_1206_3216Metric_Pad1.42x1.75mm_HandSolder (layer F.Cu)
-    (at 50.4952 22.7838 90)
+    (at 50.4698 22.7838 90)
     (descr "Capacitor SMD 1206 (3216 Metric), square (rectangular) end terminal, IPC_7351 nominal with elongated pad for handsoldering. (Body size source: http://www.tortai-tech.com/upload/download/2011102023233369053.pdf), generated with kicad-footprint-generator")
     (tags "capacitor handsolder")
@@
   )
   (module Capacitor_SMD:C_0805_2012Metric_Pad1.15x1.40mm_HandSolder (layer F.Cu)
-    (at 46.8122 27.2288 90)
+    (at 46.863 28.067 90)
     (descr "Capacitor SMD 0805 (2012 Metric), square (rectangular) end terminal, IPC_7351 nominal with elongated pad for handsoldering. (Body size source: https://docs.google.com/spreadsheets/d/1BsfQQcO9C6DZCsRaXUlFlo91Tg2WpOkGARC1WS5S8t0/edit?usp=sharing), generated with kicad-footprint-generator")
     (tags "capacitor handsolder")
@@
   (gr_line (start 20 20) (end 79.81 20) (layer Edge.Cuts) (width 0.05))
   (gr_line (start 20 20) (end 20 37.78) (layer Edge.Cuts) (width 0.05))
+  (segment (start 50.4698 26.5795) (end 48.8839 26.5795) (width 0.5) (layer F.Cu) (net 6))
+  (segment (start 48.4214 27.042) (end 46.863 27.042) (width 0.5) (layer F.Cu) (net 6))
+  (segment (start 48.8839 26.5795) (end 48.4214 27.042) (width 0.5) (layer F.Cu) (net 6))
+  (segment (start 49.0815 21.8096) (end 46.863 21.8096) (width 0.5) (layer F.Cu) (net 6))
+  (segment (start 50.4698 21.2963) (end 49.5948 21.2963) (width 0.5) (layer F.Cu) (net 6))
+  (segment (start 49.5948 21.2963) (end 49.0815 21.8096) (width 0.5) (layer F.Cu) (net 6))
+  (segment (start 54.3299 21.2963) (end 55.397 22.3634) (width 0.5) (layer F.Cu) (net 6))
+  (segment (start 50.4698 21.2963) (end 54.3299 21.2963) (width 0.5) (layer F.Cu) (net 6))
+  (segment (start 52.7862 30.8952) (end 53.6078 30.0736) (width 0.5) (layer F.Cu) (net 6))
+  (segment (start 52.7862 32.2202) (end 52.7862 30.8952) (width 0.5) (layer F.Cu) (net 6))
+  (segment (start 53.6078 30.0736) (end 55.3466 30.0736) (width 0.5) (layer F.Cu) (net 6))
+  (segment (start 55.3466 30.0736) (end 57.4802 32.2072) (width 0.5) (layer F.Cu) (net 6))
+  (segment (start 57.4802 32.2072) (end 57.4802 34.5948) (width 0.5) (layer F.Cu) (net 6))
+  (segment (start 57.4802 34.5948) (end 59.055 36.1696) (width 0.5) (layer F.Cu) (net 6))
+  (segment (start 59.055 36.1696) (end 68.58 36.1696) (width 0.5) (layer F.Cu) (net 6))
+  (segment (start 68.58 36.1696) (end 69.9008 34.8488) (width 0.5) (layer F.Cu) (net 6))
+  (segment (start 69.9008 33.4824) (end 69.8956 33.4772) (width 0.5) (layer F.Cu) (net 6))
+  (segment (start 69.9008 34.8488) (end 69.9008 33.4824) (width 0.5) (layer F.Cu) (net 6))
+  (via (at 53.1368 29.21) (size 0.8) (drill 0.4) (layers F.Cu B.Cu) (net 6))
+  (segment (start 53.6078 30.0736) (end 53.6078 29.681) (width 0.5) (layer F.Cu) (net 6))
+  (segment (start 53.6078 29.681) (end 53.1368 29.21) (width 0.5) (layer F.Cu) (net 6))
+  (segment (start 53.1368 29.21) (end 53.1368 27.0002) (width 0.5) (layer B.Cu) (net 6))
+  (via (at 52.451 26.6446) (size 0.8) (drill 0.4) (layers F.Cu B.Cu) (net 6))
+  (segment (start 53.1368 27.0002) (end 52.7812 26.6446) (width 0.5) (layer B.Cu) (net 6))
+  (segment (start 52.7812 26.6446) (end 52.451 26.6446) (width 0.5) (layer B.Cu) (net 6))
+  (segment (start 50.5349 26.6446) (end 50.4698 26.5795) (width 0.5) (layer F.Cu) (net 6))
+  (segment (start 52.451 26.6446) (end 50.5349 26.6446) (width 0.5) (layer F.Cu) (net 6))
+  (segment (start 50.1862 29.8381) (end 50.4698 29.5545) (width 0.5) (layer F.Cu) (net 7))
+  (segment (start 50.1862 32.2202) (end 50.1862 29.8381) (width 0.5) (layer F.Cu) (net 7))
+  (segment (start 50.4698 29.5545) (end 49.1125 29.5545) (width 0.5) (layer F.Cu) (net 7))
+  (segment (start 48.65 29.092) (end 46.863 29.092) (width 0.5) (layer F.Cu) (net 7))
+  (segment (start 49.1125 29.5545) (end 48.65 29.092) (width 0.5) (layer F.Cu) (net 7))
+  (segment (start 51.3448 29.5545) (end 52.705 28.1943) (width 0.5) (layer F.Cu) (net 7))
+  (segment (start 50.4698 29.5545) (end 51.3448 29.5545) (width 0.5) (layer F.Cu) (net 7))
+  (segment (start 52.705 28.1943) (end 52.705 27.9146) (width 0.5) (layer F.Cu) (net 7))
+  (segment (start 53.6562 26.9634) (end 55.397 26.9634) (width 0.5) (layer F.Cu) (net 7))
+  (segment (start 52.705 27.9146) (end 53.6562 26.9634) (width 0.5) (layer F.Cu) (net 7))
+  (segment (start 66.3956 31.7772) (end 64.692 30.0736) (width 0.5) (layer F.Cu) (net 7))
+  (segment (start 66.3956 33.4772) (end 66.3956 31.7772) (width 0.5) (layer F.Cu) (net 7))
+  (segment (start 64.692 30.0736) (end 57.1246 30.0736) (width 0.5) (layer F.Cu) (net 7))
+  (segment (start 55.397 28.346) (end 55.397 26.9634) (width 0.5) (layer F.Cu) (net 7))
+  (segment (start 57.1246 30.0736) (end 55.397 28.346) (width 0.5) (layer F.Cu) (net 7))
+  (segment (start 61.697 24.6634) (end 55.397 24.6634) (width 0.5) (layer F.Cu) (net 8))
+  (segment (start 50.8873 24.6634) (end 50.4952 24.2713) (width 0.5) (layer F.Cu) (net 8))
+  (segment (start 49.5948 24.2713) (end 49.1741 23.8506) (width 0.5) (layer F.Cu) (net 8))
+  (segment (start 50.4698 24.2713) (end 49.5948 24.2713) (width 0.5) (layer F.Cu) (net 8))
+  (segment (start 49.1651 23.8596) (end 46.863 23.8596) (width 0.5) (layer F.Cu) (net 8))
+  (segment (start 49.1741 23.8506) (end 49.1651 23.8596) (width 0.5) (layer F.Cu) (net 8))
+  (segment (start 53.5049 24.2713) (end 50.4698 24.2713) (width 0.5) (layer F.Cu) (net 8))
+  (segment (start 55.397 24.6634) (end 53.897 24.6634) (width 0.5) (layer F.Cu) (net 8))
+  (segment (start 53.897 24.6634) (end 53.5049 24.2713) (width 0.5) (layer F.Cu) (net 8))
 )

Commit message: single panel
Parts:
- removed J2, J3: Conn_01x01_Male, Connector_Wire:SolderWirePad_1x01_Drill1mm
- moved J0 28.9 mm to (70.9, 23.8)
- moved J1 26.8 mm to (30.3, 23.8)
- moved D1 6.96 mm to (41.2, 28.5)
- moved R1 5.07 mm to (41.2, 24.5)
Connections:
- D1 pad 1: Net-(C1-Pad2) -> Net-(D1-Pad1)
- D1 pad 2: Net-(D1-Pad2) -> Net-(C3-Pad1)
- R1 pad 1: Net-(C3-Pad1) -> Net-(D1-Pad1)
- R1 pad 2: Net-(D1-Pad2) -> Net-(C1-Pad2)
Routing:
- net Net-(C3-Pad1): track 15.7 -> 48.4 mm
- net Net-(C1-Pad1): track 28.2 -> 59.9 mm
- net Net-(C1-Pad2): track 43.7 -> 70.0 mm
- net Net-(D1-Pad1): track 0.00 -> 4.00 mm
- added copper zone on B.Cu, net Net-(J0-Pad1)
- added copper zone on F.Cu, net Net-(J0-Pad1)

Commit message: fixed missing routed trace
Parts:
- added REF**: OSHW-Symbol_6.7x6mm_Copper, Symbol:OSHW-Symbol_6.7x6mm_Copper, B.Cu at (64.2, 27.1)
- added REF**: OSHW-Symbol_6.7x6mm_Copper, Symbol:OSHW-Symbol_6.7x6mm_Copper, F.Cu at (72.1, 28.7)
- added REF**: OSHW-Symbol_6.7x6mm_SilkScreen, Symbol:OSHW-Symbol_6.7x6mm_SilkScreen, B.Cu at (25.9, 28.7)
- added REF**: OSHW-Symbol_6.7x6mm_SilkScreen, Symbol:OSHW-Symbol_6.7x6mm_SilkScreen, F.Cu at (41.1, 34.6)
Routing:
- net Net-(C1-Pad2): track 70.0 -> 81.6 mm, vias 2 -> 4
Other:
- board text added: "D02_ELECTRONIC"
