File: C_BREAKOUTS/C06/C06.kicad_pcb (KiCad board)
At the start: 2 copper layers, 48.3 x 27.9 mm, 40 parts, among them J1 Conn_01x02_Female, J10 Conn_01x02_Female, J11 Conn_01x02_Female, J12 Conn_01x02_Female, J13 Conn_01x02_Female, J14 Conn_01x02_Female, J15 Conn_01x02_Female, J16 Conn_01x02_Female, J17 Conn_01x02_Female, J18 Conn_01x02_Female, J19 Conn_01x02_Female, J2 Conn_01x02_Female, J20 Conn_01x02_Female, J21 Conn_01x02_Female, J22 Conn_01x02_Female, J23 Conn_01x02_Female, J24 Conn_01x02_Female, J25 Conn_01x02_Female, J26 Conn_01x02_Female, J27 Conn_01x04_Female, J28 Conn_01x04_Female, J29 Conn_01x04_Female, J3 Conn_01x02_Female, J30 Conn_01x04_Female, J31 Conn_01x04_Female, J32 Conn_01x04_Female, J33 Conn_01x04_Female, J34 Conn_01x04_Female, J35 Conn_01x04_Female, J36 Conn_01x04_Female, J4 Conn_01x07_Female, J5 Conn_01x07_Female, J6 Conn_01x02_Female, J7 Conn_01x09_Female, J8 Conn_01x09_Female, J9 Conn_01x02_Female

Commit message: all traces routed
Routing:
- net Net-(J8-Pad1): track 0.00 -> 40.6 mm
- net Net-(J7-Pad1): track 0.00 -> 40.6 mm
- net Net-(J1-Pad1): track 0.00 -> 17.3 mm
- net Net-(J3-Pad1): track 0.00 -> 17.3 mm
- net Net-(J15-Pad1): track 0.00 -> 17.3 mm
- net Net-(J20-Pad1): track 0.00 -> 17.3 mm
- net Net-(J2-Pad1): track 0.00 -> 16.5 mm
- net Net-(J14-Pad1): track 0.00 -> 16.5 mm
- net Net-(J5-Pad6): track 0.00 -> 16.5 mm
- net Net-(J19-Pad1): track 0.00 -> 16.5 mm
- net Net-(J13-Pad1): track 0.00 -> 15.7 mm
- net Net-(J11-Pad1): track 0.00 -> 15.7 mm
- net Net-(J18-Pad1): track 0.00 -> 15.7 mm
- net Net-(J16-Pad1): track 0.00 -> 15.7 mm
- net Net-(J31-Pad1): track 0.00 -> 15.2 mm
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Other:
- net class Default: trace_width 0.25 -> 0.75
- board text added: "C06_BREAKOUT"

Commit message: single gerber
Parts:
- added J37: Conn_01x01_Male, Connector_Wire:SolderWirePad_1x01_Drill1mm, F.Cu at (29.3, 23.3)
- added J38: Conn_01x01_Male, Connector_Wire:SolderWirePad_1x01_Drill1mm, F.Cu at (29.3, 44.6)
- added J39: Conn_01x01_Male, Connector_Wire:SolderWirePad_1x01_Drill1mm, F.Cu at (58.9, 23.3)
- added J40: Conn_01x01_Male, Connector_Wire:SolderWirePad_1x01_Drill1mm, F.Cu at (58.9, 44.6)
Routing:
- added copper zone on B.Cu, net Net-(J37-Pad1)
- added copper zone on F.Cu, net Net-(J37-Pad1)
Changed lines of the file:
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@@
     (tracks 188)
     (zones 0)
-    (modules 40)
-    (nets 35)
+    (modules 44)
+    (nets 36)
   )
   (page A4)
@@
     (visible_elements FFFFFF7F)
     (pcbplotparams
-      (layerselection 0x010fc_ffffffff)
+      (layerselection 0x010f0_ffffffff)
       (usegerberextensions false)
       (usegerberattributes false)
@@
       (outputformat 1)
       (mirror false)
-      (drillshape 1)
+      (drillshape 0)
       (scaleselection 1)
-      (outputdirectory ""))
+      (outputdirectory "gerber/single/"))
   )
   (net 0 "")
@@
   (net 33 "Net-(J35-Pad1)")
   (net 34 "Net-(J36-Pad1)")
+  (net 35 "Net-(J37-Pad1)")
   (net_class Default "This is the default net class."
     (clearance 0.2)
@@
     (add_net "Net-(J35-Pad1)")
     (add_net "Net-(J36-Pad1)")
+    (add_net "Net-(J37-Pad1)")
     (add_net "Net-(J5-Pad6)")
     (add_net "Net-(J7-Pad1)")
     (add_net "Net-(J8-Pad1)")
     (add_net "Net-(J9-Pad1)")
+  )
+  (module Connector_Wire:SolderWirePad_1x01_Drill1mm (layer F.Cu)
+    (at 58.9484 44.6228)
+    (descr "Wire solder connection")
+    (tags connector)
+    (attr virtual)
+    (fp_text reference J40 (at 0 -3.81) (layer F.SilkS) hide
+      (effects (font (size 1 1) (thickness 0.15)))
+    )
+    (fp_text value Conn_01x01_Male (at 0 3.175) (layer F.Fab)
+      (effects (font (size 1 1) (thickness 0.15)))
+    )
+    (fp_line (start 1.75 1.75) (end -1.75 1.75) (layer F.CrtYd) (width 0.05))
+    (fp_line (start 1.75 1.75) (end 1.75 -1.75) (layer F.CrtYd) (width 0.05))
+    (fp_line (start -1.75 -1.75) (end -1.75 1.75) (layer F.CrtYd) (width 0.05))
+    (fp_line (start -1.75 -1.75) (end 1.75 -1.75) (layer F.CrtYd) (width 0.05))
+    (fp_text user %R (at 0 0) (layer F.Fab)
+      (effects (font (size 1 1) (thickness 0.15)))
+    )
+    (pad 1 thru_hole circle (at 0 0) (size 2.49936 2.49936) (drill 1.00076) (layers *.Cu *.Mask)
+      (net 35 "Net-(J37-Pad1)"))
+  )
+  (module Connector_Wire:SolderWirePad_1x01_Drill1mm (layer F.Cu)
+    (at 58.9484 23.3172)
+    (descr "Wire solder connection")
+    (tags connector)
+    (attr virtual)
+    (fp_text reference J39 (at 0 -3.81) (layer F.SilkS) hide
+      (effects (font (size 1 1) (thickness 0.15)))
+    )
+    (fp_text value Conn_01x01_Male (at 0 3.175) (layer F.Fab)
+      (effects (font (size 1 1) (thickness 0.15)))
+    )
+    (fp_line (start 1.75 1.75) (end -1.75 1.75) (layer F.CrtYd) (width 0.05))
+    (fp_line (start 1.75 1.75) (end 1.75 -1.75) (layer F.CrtYd) (width 0.05))
+    (fp_line (start -1.75 -1.75) (end -1.75 1.75) (layer F.CrtYd) (width 0.05))
+    (fp_line (start -1.75 -1.75) (end 1.75 -1.75) (layer F.CrtYd) (width 0.05))
+    (fp_text user %R (at 0 0) (layer F.Fab)
+      (effects (font (size 1 1) (thickness 0.15)))
+    )
+    (pad 1 thru_hole circle (at 0 0) (size 2.49936 2.49936) (drill 1.00076) (layers *.Cu *.Mask)
+      (net 35 "Net-(J37-Pad1)"))
+  )
+  (module Connector_Wire:SolderWirePad_1x01_Drill1mm (layer F.Cu)
+    (at 29.3116 44.6228)
+    (descr "Wire solder connection")
+    (tags connector)
+    (attr virtual)
+    (fp_text reference J38 (at 0 -3.81) (layer F.SilkS) hide
+      (effects (font (size 1 1) (thickness 0.15)))
+    )
+    (fp_text value Conn_01x01_Male (at 0 3.175) (layer F.Fab)
+      (effects (font (size 1 1) (thickness 0.15)))
+    )
+    (fp_line (start 1.75 1.75) (end -1.75 1.75) (layer F.CrtYd) (width 0.05))
+    (fp_line (start 1.75 1.75) (end 1.75 -1.75) (layer F.CrtYd) (width 0.05))
+    (fp_line (start -1.75 -1.75) (end -1.75 1.75) (layer F.CrtYd) (width 0.05))
+    (fp_line (start -1.75 -1.75) (end 1.75 -1.75) (layer F.CrtYd) (width 0.05))
+    (fp_text user %R (at 0 0) (layer F.Fab)
+      (effects (font (size 1 1) (thickness 0.15)))
+    )
+    (pad 1 thru_hole circle (at 0 0) (size 2.49936 2.49936) (drill 1.00076) (layers *.Cu *.Mask)
+      (net 35 "Net-(J37-Pad1)"))
+  )
+  (module Connector_Wire:SolderWirePad_1x01_Drill1mm (layer F.Cu)
+    (at 29.3116 23.3172)
+    (descr "Wire solder connection")
+    (tags connector)
+    (attr virtual)
+    (fp_text reference J37 (at 0 -3.81) (layer F.SilkS) hide
+      (effects (font (size 1 1) (thickness 0.15)))
+    )
+    (fp_text value Conn_01x01_Male (at 0 3.175) (layer F.Fab)
+      (effects (font (size 1 1) (thickness 0.15)))
+    )
+    (fp_line (start 1.75 1.75) (end -1.75 1.75) (layer F.CrtYd) (width 0.05))
+    (fp_line (start 1.75 1.75) (end 1.75 -1.75) (layer F.CrtYd) (width 0.05))
+    (fp_line (start -1.75 -1.75) (end -1.75 1.75) (layer F.CrtYd) (width 0.05))
+    (fp_line (start -1.75 -1.75) (end 1.75 -1.75) (layer F.CrtYd) (width 0.05))
+    (fp_text user %R (at 0 0) (layer F.Fab)
+      (effects (font (size 1 1) (thickness 0.15)))
+    )
+    (pad 1 thru_hole circle (at 0 0) (size 2.49936 2.49936) (drill 1.00076) (layers *.Cu *.Mask)
+      (net 35 "Net-(J37-Pad1)"))
   )
   (module Connector_PinHeader_2.54mm:PinHeader_1x04_P2.54mm_Vertical (layer F.Cu)
@@
   (segment (start 49.21 40.32) (end 49.21 42.86) (width 0.75) (layer B.Cu) (net 34))
   (segment (start 49.21 42.86) (end 49.21 45.4) (width 0.75) (layer B.Cu) (net 34))
+  (zone (net 35) (net_name "Net-(J37-Pad1)") (layer F.Cu) (hatch edge 0.508)
+    (connect_pads (clearance 0.508))
+    (min_thickness 0.254)
+    (fill yes (arc_segments 32) (thermal_gap 0.508) (thermal_bridge_width 0.508))
+    (polygon
+      (pts
+        (xy 67.7164 20.5232) (xy 67.7418 47.371) (xy 20.5232 47.4726) (xy 20.574 20.574)
+      )
+    )
+  )
+  (zone (net 35) (net_name "Net-(J37-Pad1)") (layer B.Cu) (hatch edge 0.508)
+    (connect_pads (clearance 0.508))
+    (min_thickness 0.254)
+    (fill yes (arc_segments 32) (thermal_gap 0.508) (thermal_bridge_width 0.508))
+    (polygon
+      (pts
+        (xy 67.7418 20.4978) (xy 67.7164 47.371) (xy 20.5232 47.4726) (xy 20.574 20.574)
+      )
+    )
+  )
 )
