File: D_ELECTRONICS/D05/D05.kicad_pcb (KiCad board)
At the start: 2 copper layers, 48.3 x 17.8 mm, 26 parts, among them J0 Conn_01x01_Male, J1 Conn_01x01_Male, J2 Conn_01x01_Male, J3 Conn_01x01_Male, J4 Conn_01x10_Female, J6 Conn_01x10_Female

Commit message: all traces routed
Parts:
- removed HZ0, HZ1, HZ10, HZ11, HZ12, HZ13, HZ14, HZ15, HZ2, HZ3, HZ4, HZ5, HZ6, HZ7, HZ8, HZ9: MountingHole, MountingHole:MountingHole_3mm
- removed J2, J3: Conn_01x01_Male, Connector_Wire:SolderWirePad_1x01_Drill1mm
- removed J6: Conn_01x10_Female, TerminalBlock_4Ucon:TerminalBlock_4Ucon_1x10_P3.50mm_Horizontal
- added J5: Conn_01x09_Female, TerminalBlock_4Ucon:TerminalBlock_4Ucon_1x09_P3.50mm_Horizontal, F.Cu at (30.1, 33.8)
- added R1: R, Resistor_THT:R_Axial_DIN0204_L3.6mm_D1.6mm_P2.54mm_Vertical, F.Cu at (39.9, 26.8)
- added R11: R, Resistor_SMD:R_0805_2012Metric_Pad1.15x1.40mm_HandSolder, F.Cu at (40.7, 28.9)
- added R2: R, Resistor_THT:R_Axial_DIN0204_L3.6mm_D1.6mm_P2.54mm_Vertical, F.Cu at (28.3, 24.5)
- added R22: R, Resistor_SMD:R_0805_2012Metric_Pad1.15x1.40mm_HandSolder, F.Cu at (28.4, 26.7)
- added R3: R, Resistor_THT:R_Axial_DIN0204_L3.6mm_D1.6mm_P2.54mm_Vertical, F.Cu at (33.0, 24.5)
- added R33: R, Resistor_SMD:R_0805_2012Metric_Pad1.15x1.40mm_HandSolder, F.Cu at (32.2, 26.7)
- added R4: R, Resistor_THT:R_Axial_DIN0204_L3.6mm_D1.6mm_P2.54mm_Vertical, F.Cu at (37.6, 24.5)
- added R44: R, Resistor_SMD:R_0805_2012Metric_Pad1.15x1.40mm_HandSolder, F.Cu at (36.0, 26.7)
- moved J0 213.3 mm to (23.8, 28.9)
- moved J1 170.8 mm to (64.5, 28.9)
Routing:
- net Net-(J4-Pad8): track 0.00 -> 30.6 mm
- net Net-(J5-Pad2): track 0.00 -> 27.1 mm
- net Net-(J4-Pad1): track 0.00 -> 26.8 mm
- net Net-(J4-Pad2): track 0.00 -> 26.0 mm
- net Net-(J4-Pad5): track 0.00 -> 25.7 mm
- net Net-(J4-Pad3): track 0.00 -> 25.2 mm
- net Net-(J4-Pad4): track 0.00 -> 24.9 mm
- net Net-(J5-Pad1): track 0.00 -> 21.7 mm
- net Net-(J5-Pad3): track 0.00 -> 16.3 mm
- net Net-(J4-Pad7): track 0.00 -> 12.5 mm
- added copper zone on B.Cu, net Net-(J0-Pad1)
- added copper zone on F.Cu, net Net-(J0-Pad1)
Other:
- net class Default: trace_width 0.25 -> 0.75
