File: D_ELECTRONICS/D05/D05.kicad_pcb (KiCad board)
At the start: 2 copper layers, 48.3 x 17.8 mm, 16 parts, among them J0 Conn_01x01_Male, J1 Conn_01x01_Male, J4 Conn_01x10_Female, J5 Conn_01x09_Female

Commit message: missing part number
Parts:
- added REF**: OSHW-Symbol_6.7x6mm_Copper, Symbol:OSHW-Symbol_6.7x6mm_Copper, B.Cu at (59.9, 28.8)
- added REF**: OSHW-Symbol_6.7x6mm_SilkScreen, Symbol:OSHW-Symbol_6.7x6mm_SilkScreen, F.Cu at (59.6, 24.6)
Other:
- board text added: "D05_ELE"
