File: a-backplates/a06/a06.kicad_pcb (KiCad board)
At the start: 2 copper layers, 90 x 58 mm, 9 parts, among them J1 Conn_01x01_Male, J2 Conn_01x01_Male

Commit message: backplate A06 finished pcb
Parts:
- added REF**: OSHW-Symbol_6.7x6mm_Copper, Symbol:OSHW-Symbol_6.7x6mm_Copper, F.Cu at (139.7, 138.9)
- added REF**: OSHW-Symbol_6.7x6mm_SilkScreen, Symbol:OSHW-Symbol_6.7x6mm_SilkScreen, B.Cu at (170.4, 118.4)
- added REF**: OSHW-Symbol_6.7x6mm_Copper, Symbol:OSHW-Symbol_6.7x6mm_Copper, B.Cu at (170.4, 138.9)
- added REF**: OSHW-Symbol_6.7x6mm_SilkScreen, Symbol:OSHW-Symbol_6.7x6mm_SilkScreen, F.Cu at (139.7, 118.4)
- added REF**1: MountingHole_3mm, MountingHole:MountingHole_3mm, F.Cu at (114.5, 103.6)
- added REF**10: MountingHole_3mm, MountingHole:MountingHole_3mm, F.Cu at (114.5, 113.8)
- added REF**11: MountingHole_3mm, MountingHole:MountingHole_3mm, F.Cu at (124.7, 113.8)
- added REF**12: MountingHole_3mm, MountingHole:MountingHole_3mm, F.Cu at (134.8, 113.8)
- added REF**13: MountingHole_3mm, MountingHole:MountingHole_3mm, F.Cu at (145.0, 113.8)
- added REF**14: MountingHole_3mm, MountingHole:MountingHole_3mm, F.Cu at (155.2, 113.8)
- added REF**15: MountingHole_3mm, MountingHole:MountingHole_3mm, F.Cu at (165.3, 113.8)
- added REF**16: MountingHole_3mm, MountingHole:MountingHole_3mm, F.Cu at (175.5, 113.8)
- added REF**17: MountingHole_3mm, MountingHole:MountingHole_3mm, F.Cu at (185.6, 113.8)
- added REF**18: MountingHole_3mm, MountingHole:MountingHole_3mm, F.Cu at (104.4, 123.9)
- added REF**19: MountingHole_3mm, MountingHole:MountingHole_3mm, F.Cu at (114.5, 123.9)
- added REF**2: MountingHole_3mm, MountingHole:MountingHole_3mm, F.Cu at (124.7, 103.6)
- added REF**20: MountingHole_3mm, MountingHole:MountingHole_3mm, F.Cu at (124.7, 123.9)
- added REF**21: MountingHole_3mm, MountingHole:MountingHole_3mm, F.Cu at (134.8, 123.9)
- added REF**22: MountingHole_3mm, MountingHole:MountingHole_3mm, F.Cu at (145.0, 123.9)
- added REF**23: MountingHole_3mm, MountingHole:MountingHole_3mm, F.Cu at (155.2, 123.9)
- added REF**24: MountingHole_3mm, MountingHole:MountingHole_3mm, F.Cu at (165.3, 123.9)
- added REF**25: MountingHole_3mm, MountingHole:MountingHole_3mm, F.Cu at (175.5, 123.9)
- added REF**26: MountingHole_3mm, MountingHole:MountingHole_3mm, F.Cu at (185.6, 123.9)
- added REF**27: MountingHole_3mm, MountingHole:MountingHole_3mm, F.Cu at (104.4, 134.1)
- added REF**28: MountingHole_3mm, MountingHole:MountingHole_3mm, F.Cu at (114.5, 134.1)
- added REF**29: MountingHole_3mm, MountingHole:MountingHole_3mm, F.Cu at (124.7, 134.1)
- added REF**3: MountingHole_3mm, MountingHole:MountingHole_3mm, F.Cu at (134.8, 103.6)
- added REF**30: MountingHole_3mm, MountingHole:MountingHole_3mm, F.Cu at (134.8, 134.1)
- added REF**31: MountingHole_3mm, MountingHole:MountingHole_3mm, F.Cu at (145.0, 134.1)
- added REF**32: MountingHole_3mm, MountingHole:MountingHole_3mm, F.Cu at (155.2, 134.1)
- added REF**33: MountingHole_3mm, MountingHole:MountingHole_3mm, F.Cu at (165.3, 134.1)
- added REF**34: MountingHole_3mm, MountingHole:MountingHole_3mm, F.Cu at (175.5, 134.1)
- added REF**35: MountingHole_3mm, MountingHole:MountingHole_3mm, F.Cu at (185.6, 134.1)
- added REF**36: MountingHole_3mm, MountingHole:MountingHole_3mm, F.Cu at (104.4, 144.2)
- added REF**37: MountingHole_3mm, MountingHole:MountingHole_3mm, F.Cu at (114.5, 144.2)
- added REF**38: MountingHole_3mm, MountingHole:MountingHole_3mm, F.Cu at (124.7, 144.2)
- added REF**39: MountingHole_3mm, MountingHole:MountingHole_3mm, F.Cu at (134.8, 144.2)
- added REF**4: MountingHole_3mm, MountingHole:MountingHole_3mm, F.Cu at (145.0, 103.6)
- added REF**40: MountingHole_3mm, MountingHole:MountingHole_3mm, F.Cu at (145.0, 144.2)
- added REF**41: MountingHole_3mm, MountingHole:MountingHole_3mm, F.Cu at (155.2, 144.2)
- added REF**42: MountingHole_3mm, MountingHole:MountingHole_3mm, F.Cu at (165.3, 144.2)
- added REF**43: MountingHole_3mm, MountingHole:MountingHole_3mm, F.Cu at (175.5, 144.2)
- added REF**44: MountingHole_3mm, MountingHole:MountingHole_3mm, F.Cu at (185.6, 144.2)
- added REF**46: MountingHole_3mm, MountingHole:MountingHole_3mm, F.Cu at (114.5, 154.4)
- added REF**48: MountingHole_3mm, MountingHole:MountingHole_3mm, F.Cu at (134.8, 154.4)
- added REF**49: MountingHole_3mm, MountingHole:MountingHole_3mm, F.Cu at (145.0, 154.4)
- added REF**5: MountingHole_3mm, MountingHole:MountingHole_3mm, F.Cu at (155.2, 103.6)
- added REF**50: MountingHole_3mm, MountingHole:MountingHole_3mm, F.Cu at (155.2, 154.4)
- added REF**52: MountingHole_3mm, MountingHole:MountingHole_3mm, F.Cu at (175.5, 154.4)
- added REF**7: MountingHole_3mm, MountingHole:MountingHole_3mm, F.Cu at (175.5, 103.6)
- moved J1 35.7 mm to (185.6, 118.8)
- moved J2 28.3 mm to (104.4, 139.2)
Routing:
- added copper zone on F.Cu, net (none)
- added copper zone on B.Cu, net Net-(J1-Pad1)
Other:
- board text added: "A06_BACKPLATE"
