File: c-breakouts/c12/C12.sch (KiCad schematic (older format))
At the start: 12 parts, among them J0 Conn_01x01_Male, J1 Conn_01x01_Male, J2 Conn_01x01_Male, J3 Conn_01x01_Male, J4 Conn_01x08_Female, J5 Conn_01x08_Female, J6 Conn_01x08_Female, J7 Conn_01x08_Female

Commit message: expanded breakout C012 to wemos esp32
Parts:
- removed J2, J3: Conn_01x01_Male, Connector_Wire:SolderWirePad_1x01_Drill1mm, symbol Connector:Conn_01x01_Male
- removed J4, J5: Conn_01x08_Female, TerminalBlock_4Ucon:TerminalBlock_4Ucon_1x08_P3.50mm_Horizontal, symbol Connector:Conn_01x08_Female
- removed J6, J7: Conn_01x08_Female, Connector_PinSocket_2.54mm:PinSocket_1x08_P2.54mm_Vertical, symbol Connector:Conn_01x08_Female
- added J1, J2, J3, J4: Conn_01x10_Female, Connector_PinHeader_2.54mm:PinHeader_1x10_P2.54mm_Vertical, symbol Connector:Conn_01x10_Female
- added J5, J6: Conn_01x10_Female, TerminalBlock_4Ucon:TerminalBlock_4Ucon_1x10_P3.50mm_Vertical, symbol Connector:Conn_01x10_Female
- added JP1, JP10, JP2, JP21, JP22, JP23, JP24, JP25, JP26, JP27, JP28, JP29, JP3, JP30, JP4, JP5, JP6, JP7, JP8, JP9: SolderJumper_2_Bridged, Jumper:SolderJumper-2_P1.3mm_Bridged_RoundedPad1.0x1.5mm, symbol Jumper:SolderJumper_2_Bridged
- added JP11, JP12, JP13, JP14, JP15, JP16, JP17, JP18, JP19, JP20, JP31, JP32, JP33, JP34, JP35, JP36, JP37, JP38, JP39, JP40: SolderJumper_2_Open, Jumper:SolderJumper-2_P1.3mm_Open_RoundedPad1.0x1.5mm, symbol Jumper:SolderJumper_2_Open
- renumbered J0 to J10, J1 to J11
Connections:
- net labels removed: ENCLOSURE_MOUNT_HOLES
- wire segments 23 -> 113
