File: a-backplates/a07/A07.kicad_pcb (KiCad board)
At the start: 2 copper layers, 49 x 47 mm, 28 parts, among them J0 Conn_01x01_Male, J1 Conn_01x01_Male, J2 Conn_01x01_Male, J3 Conn_01x01_Male

Commit message: pictures for A07 orange pi plate
Other:
- rule pad_to_mask_clearance: 0.051 -> 0
Changed lines of the file:
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@@
   )
   (setup
-    (pad_to_mask_clearance 0.051)
-    (solder_mask_min_width 0.25)
+    (stackup
+      (layer "F.SilkS" (type "Top Silk Screen"))
+      (layer "F.Paste" (type "Top Solder Paste"))
+      (layer "F.Mask" (type "Top Solder Mask") (thickness 0.01))
+      (layer "F.Cu" (type "copper") (thickness 0.035))
+      (layer "dielectric 1" (type "core") (thickness 1.51) (material "FR4") (epsilon_r 4.5) (loss_tangent 0.02))
+      (layer "B.Cu" (type "copper") (thickness 0.035))
+      (layer "B.Mask" (type "Bottom Solder Mask") (thickness 0.01))
+      (layer "B.Paste" (type "Bottom Solder Paste"))
+      (layer "B.SilkS" (type "Bottom Silk Screen"))
+      (copper_finish "None")
+      (dielectric_constraints no)
+    )
+    (pad_to_mask_clearance 0)
     (pcbplotparams
       (layerselection 0x00010f0_ffffffff)
@@
       (svguseinch false)
       (svgprecision 6)
-      (excludeedgelayer true)
+      (excludeedgelayer false)
       (plotframeref false)
       (viasonmask false)
